File: circuit/Altair Nexus Driver Module.kicad_sch (KiCad schematic)
At the start: 0 parts

Commit message: feat: add initial KiCad schematic, project files, and history tracking for Altair Nexus Driver Module
Parts:
- added U1: NUCLEOH723ZG, NUCLEOH723ZG:MODULE_NUCLEOH723ZG, symbol NUCLEOH723ZG:NUCLEOH723ZG
Connections:
- new net: U1.CN11_10 (NC), U1.CN11_26 (NC), U1.CN11_67 (NC)
- new net +3V3: U1.CN11_16 (3V3), U1.CN11_5 (3V3_VDD)
- new net +5V: U1.CN11_18 (5V)
- new net BUTTON: U1.CN11_23 (PC13)
- new net ENC1_CS: U1.CN12_46 (PD14)
- new net ENC2_CS: U1.CN12_48 (PD15)
- new net ENC3_CS: U1.CN12_47 (PE10)
- new net ENC4_CS: U1.CN12_49 (PE12)
- new net ENC5_A: U1.CN11_17 (PA15)
- new net ENC5_B: U1.CN12_31 (PB3)
- new net ENC6_A: U1.CN12_27 (PB4)
- new net ENC6_B: U1.CN12_29 (PB5)
- new net ENC7_A: U1.CN12_43 (PD12)
- new net ENC7_B: U1.CN12_41 (PD13)
- new net ENC8_A: U1.CN11_53 (PF0)
- new net ENC8_B: U1.CN11_51 (PF1)
- new net ETH_CRS_DV: U1.CN12_15 (PA7)
- new net ETH_MDC: U1.CN11_36 (PC1)
- new net ETH_MDIO: U1.CN12_35 (PA2)
- new net ETH_REF_CLK: U1.CN11_30 (PA1)
- new net ETH_RXD0: U1.CN12_34 (PC4)
- new net ETH_RXD1: U1.CN12_6 (PC5)
- new net ETH_TXD0: U1.CN11_68 (PG13)
- new net ETH_TXD1: U1.CN12_30 (PB13)
- new net ETH_TX_EN: U1.CN11_70 (PG11)
- new net EXT_LED1: U1.CN12_65 (PD10)
- new net EXT_LED2: U1.CN12_45 (PD11)
- new net EXT_LED3: U1.CN12_53 (PE15)
- new net FDCAN1_RX: U1.CN11_57 (PD0)
- new net FDCAN1_TX: U1.CN11_55 (PD1)
- new net FDCAN2_RX: U1.CN12_16 (PB12)
- new net FDCAN2_TX: U1.CN12_17 (PB6)
- new net GND: U1.CN11_19 (GND_CN11), U1.CN11_20 (GND_CN11), U1.CN11_22 (GND_CN11), U1.CN11_49 (GND_CN11), U1.CN11_60 (GND_CN11), U1.CN11_8 (GND_CN11), U1.CN12_20 (GND_CN12), U1.CN12_39 (GND_CN12), U1.CN12_54 (GND_CN12), U1.CN12_63 (GND_CN12), U1.CN12_9 (GND_CN12), U1.CN15_1 (GND_CN15), U1.CN15_2 (GND_CN15), U1.CN16_1 (GND_CN16), U1.CN16_2 (GND_CN16)
- new net I2C1_SCL: U1.CN12_3 (PB8)
- new net I2C1_SDA: U1.CN12_5 (PB9)
- new net I2C2_SCL: U1.CN12_25 (PB10)
- new net I2C2_SDA: U1.CN12_18 (PB11)
- new net LD1: U1.CN11_34 (PB0)
- new net LD2: U1.CN11_61 (PE1)
- new net LIMIT_SW1: U1.CN11_59 (PG0)
- new net LIMIT_SW10: U1.CN11_65 (PG12)
- new net LIMIT_SW11: U1.CN12_61 (PG14)
- new net LIMIT_SW12: U1.CN11_64 (PG15)
- new net LIMIT_SW2: U1.CN11_58 (PG1)
- new net LIMIT_SW3: U1.CN11_42 (PG2)
- new net LIMIT_SW4: U1.CN11_44 (PG3)
- new net LIMIT_SW5: U1.CN12_69 (PG4)
- new net LIMIT_SW6: U1.CN12_68 (PG5)
- new net LIMIT_SW7: U1.CN12_66 (PG8)
- new net LIMIT_SW8: U1.CN11_63 (PG9)
- new net LIMIT_SW9: U1.CN11_66 (PG10)
- new net M1_PWM1: U1.CN12_52 (PE9)
- new net M1_PWM2: U1.CN12_56 (PE11)
- new net M2_PWM1: U1.CN12_55 (PE13)
- new net M2_PWM2: U1.CN12_51 (PE14)
- new net M3_PWM1: U1.CN12_4 (PC6)
- new net M3_PWM2: U1.CN12_19 (PC7)
- new net M4_PWM1: U1.CN12_2 (PC8)
- new net M4_PWM2: U1.CN12_1 (PC9)
- new net M5_PWM1: U1.CN12_62 (PF11)
- new net M5_PWM2: U1.CN12_59 (PF12)
- new net M6_PWM1: U1.CN12_57 (PF13)
- new net M6_PWM2: U1.CN12_50 (PF14)
- new net M7_PWM1: U1.CN12_28 (PB14)
- new net M7_PWM2: U1.CN12_26 (PB15)
- new net M8_PWM1: U1.CN11_50 (PE5)
- new net M8_PWM2: U1.CN11_62 (PE6)
- new net OSC32_IN: U1.CN11_25 (PC14)
- new net OSC32_OUT: U1.CN11_27 (PC15)
- new net SERVO1: U1.CN11_28 (PA0)
- new net SERVO2: U1.CN12_37 (PA3)
- new net SERVO3: U1.CN11_54 (PF8)
- new net SERVO4: U1.CN11_56 (PF9)
- new net SERVO5: U1.CN11_9 (PF6)
- new net SERVO6: U1.CN11_11 (PF7)
- new net SOLENOID1: U1.CN11_52 (PF2)
- new net SOLENOID10: U1.CN11_48 (PE4)
- new net SOLENOID2: U1.CN12_58 (PF3)
- new net SOLENOID3: U1.CN12_38 (PF4)
- new net SOLENOID4: U1.CN12_60 (PF15)
- new net SOLENOID5: U1.CN11_4 (PD2)
- new net SOLENOID6: U1.CN11_40 (PD3)
- new net SOLENOID7: U1.CN11_39 (PD4)
- new net SOLENOID8: U1.CN11_46 (PE2)
- new net SOLENOID9: U1.CN11_47 (PE3)
- new net SPI1_MISO: U1.CN12_13 (PA6)
- new net SPI1_MOSI: U1.CN11_45 (PD7)
- new net SPI1_SCK: U1.CN12_11 (PA5)
- new net SPI3_MISO: U1.CN11_2 (PC11)
- new net SPI3_MOSI: U1.CN11_3 (PC12)
- new net SPI3_SCK: U1.CN11_1 (PC10)
- new net SWCLK: U1.CN11_15 (PA14)
- new net SWDIO: U1.CN11_13 (PA13)
- new net UART7_RX: U1.CN12_44 (PE7)
- new net UART7_TX: U1.CN12_40 (PE8)
- new net USART2_RX: U1.CN11_43 (PD6)
- new net USART2_TX: U1.CN11_41 (PD5)
- new net USART3_RX: U1.CN11_69 (PD9)
- new net USART3_TX: U1.CN12_10 (PD8)

Commit message: feat: 回路設計
Parts:
- added C1, C2, C3, C4, C5, C6, C7: 0.1u, Capacitor_SMD:C_0603_1608Metric, symbol Device:C
- added D1, D10, D11, D12, D13, D14, D15, D16, D6, D9: SS14, Diode_SMD:D_SMA, symbol Diode:SS14
- added D2, D3, D4, D5, D7, D8: LED, symbol Device:LED
- added IC1, IC2, IC3: TLP2105_F_, Library:TLP2105, symbol TLP2105_F_:TLP2105_F_
- added J1: SOLENOID1, Connector_AMASS:AMASS_XT30U-F_1x02_P5.0mm_Vertical, symbol Connector_Generic:Conn_01x02
- added J10, J6: CAN1, symbol Connector_Generic:Conn_01x02
- added J11: USART3, symbol Connector_Generic:Conn_01x04
- added J12: SPI3, symbol Connector_Generic:Conn_01x05
- added J13, J8: I2C, symbol Connector_Generic:Conn_01x05
- added J14: UART7, symbol Connector_Generic:Conn_01x04
- added J15: SOLENOID5, Connector_AMASS:AMASS_XT30U-F_1x02_P5.0mm_Vertical, symbol Connector_Generic:Conn_01x02
- added J16: SOLENOID6, Connector_AMASS:AMASS_XT30U-F_1x02_P5.0mm_Vertical, symbol Connector_Generic:Conn_01x02
- added J17, J32: TERM_EN, Connector_PinSocket_2.54mm:PinSocket_1x02_P2.54mm_Vertical, symbol Connector_Generic:Conn_01x02
- added J18: motor1, symbol Connector_Generic:Conn_01x04
- added J19: motor5, symbol Connector_Generic:Conn_01x04
- added J2: SOLENOID2, Connector_AMASS:AMASS_XT30U-F_1x02_P5.0mm_Vertical, symbol Connector_Generic:Conn_01x02
- added J20: Incremental encoder1, symbol Connector_Generic:Conn_01x04
- added J21: SOLENOID7, Connector_AMASS:AMASS_XT30U-F_1x02_P5.0mm_Vertical, symbol Connector_Generic:Conn_01x02
- added J22: motor2, symbol Connector_Generic:Conn_01x04
- added J23: motor6, symbol Connector_Generic:Conn_01x04
- added J24: Incremental encoder2, symbol Connector_Generic:Conn_01x04
- added J25: motor3, symbol Connector_Generic:Conn_01x04
- added J26: motor7, symbol Connector_Generic:Conn_01x04
- added J27: Incremental encoder3, symbol Connector_Generic:Conn_01x04
- added J28: SOLENOID8, Connector_AMASS:AMASS_XT30U-F_1x02_P5.0mm_Vertical, symbol Connector_Generic:Conn_01x02
- added J29: motor4, symbol Connector_Generic:Conn_01x04
- added J3, J4: 5V, symbol Connector_Generic:Conn_01x02
- added J30: motor8, symbol Connector_Generic:Conn_01x04
- added J31: Incremental encoder4, symbol Connector_Generic:Conn_01x04
- added J33: SOLENOID9, Connector_AMASS:AMASS_XT30U-F_1x02_P5.0mm_Vertical, symbol Connector_Generic:Conn_01x02
- added J34: LIMIT_SW1, symbol Connector_Generic:Conn_01x02
- added J35: Absolute Rotary Encoder1, symbol Connector_Generic:Conn_01x06
- added J36: LIMIT_SW2, symbol Connector_Generic:Conn_01x02
- added J37: LIMIT_SW3, symbol Connector_Generic:Conn_01x02
- added J38: SOLENOID10, Connector_AMASS:AMASS_XT30U-F_1x02_P5.0mm_Vertical, symbol Connector_Generic:Conn_01x02
- added J39: LIMIT_SW4, symbol Connector_Generic:Conn_01x02
- added J40: Absolute Rotary Encoder2, symbol Connector_Generic:Conn_01x06
- added J41: LIMIT_SW5, symbol Connector_Generic:Conn_01x02
- added J42: LIMIT_SW6, symbol Connector_Generic:Conn_01x02
- added J43: Absolute Rotary Encoder3, symbol Connector_Generic:Conn_01x06
- added J44: LIMIT_SW7, symbol Connector_Generic:Conn_01x02
- added J45: LIMIT_SW8, symbol Connector_Generic:Conn_01x02
- added J46: LIMIT_SW9, symbol Connector_Generic:Conn_01x02
- added J47: Absolute Rotary Encoder4, symbol Connector_Generic:Conn_01x06
- added J48: LIMIT_SW10, symbol Connector_Generic:Conn_01x02
- added J49, J50: 24v, symbol Connector_Generic:Conn_01x02
- added J5: SOLENOID3, Connector_AMASS:AMASS_XT30U-F_1x02_P5.0mm_Vertical, symbol Connector_Generic:Conn_01x02
- added J51, J52: 8V, symbol Connector_Generic:Conn_01x02
- added J7: USART2, symbol Connector_Generic:Conn_01x04
- added J9: SOLENOID4, Connector_AMASS:AMASS_XT30U-F_1x02_P5.0mm_Vertical, symbol Connector_Generic:Conn_01x02
- added M1: Motor_Servo1, Connector_JST:JST_XA_S03B-XASK-1_1x03_P2.50mm_Horizontal, symbol Motor:Motor_Servo
- added M2: Motor_Servo2, Connector_JST:JST_XA_S03B-XASK-1_1x03_P2.50mm_Horizontal, symbol Motor:Motor_Servo
- added M3: Motor_Servo3, Connector_JST:JST_XA_S03B-XASK-1_1x03_P2.50mm_Horizontal, symbol Motor:Motor_Servo
- added M4: Motor_Serv4, Connector_JST:JST_XA_S03B-XASK-1_1x03_P2.50mm_Horizontal, symbol Motor:Motor_Servo
- added M5: Motor_Servo5, Connector_JST:JST_XA_S03B-XASK-1_1x03_P2.50mm_Horizontal, symbol Motor:Motor_Servo
- added M6: Motor_Servo6, Connector_JST:JST_XA_S03B-XASK-1_1x03_P2.50mm_Horizontal, symbol Motor:Motor_Servo
- added Q1, Q10, Q2, Q3, Q4, Q5, Q6, Q7, Q8, Q9: AO3400A, Package_TO_SOT_SMD:SOT-23, symbol Transistor_FET:AO3400A
- added R1, R10, R15, R20, R25, R28, R32, R35, R39, R45: 470, Resistor_SMD:R_0603_1608Metric, symbol Device:R
- added R11, R12, R16, R17, R21, R23, R26, R27, R29, R30, R33, R34, R36, R37, R4, R41, R42, R47, R49, R5: 10K, Resistor_SMD:R_0603_1608Metric, symbol Device:R
- added R13, R14, R40, R43, R44, R46, R48, R50, R51, R52, R53, R54: 4.7k, symbol Device:R
- added R18, R19, R22, R24: 3.3k, symbol Device:R
- added R2, R3, R6, R7, R8, R9: 4.7k, Resistor_SMD:R_0603_1608Metric, symbol Device:R
- added R31, R38: 120, Resistor_SMD:R_0603_1608Metric, symbol Device:R
- added SW1: SW_DPDT_x2, symbol Switch:SW_DPDT_x2
- added U1, U3, U4: TLP291-4, Package_SO:SOIC-16_4.55x10.3mm_P1.27mm, symbol Isolator:TLP291-4
- added U5, U6: MCP2562-E-SN, Package_SO:SOIC-8_3.9x4.9mm_P1.27mm, symbol Interface_CAN_LIN:MCP2562-E-SN
- renumbered U1 to U2
Connections:
- net +3V3: now also J13.1 (Pin_1), J8.1 (Pin_1), R13.2, R14.2, R18.2, R19.2, R22.2, R24.2, R40.1, R43.1, R44.1, R46.1, R48.1, R50.1, R51.1, R52.1, R53.1, R54.1
- net +5V: now also U2.CN11_6 (5V_EXT), C1.1, C3.1, J11.1 (Pin_1), J12.1 (Pin_1), J14.1 (Pin_1), J18.2 (Pin_2), J19.2 (Pin_2), J20.2 (Pin_2), J22.2 (Pin_2), J23.2 (Pin_2), J24.2 (Pin_2), J25.2 (Pin_2), J26.2 (Pin_2), J27.2 (Pin_2), J29.2 (Pin_2), J3.1 (Pin_1), J30.2 (Pin_2), J31.2 (Pin_2), J35.1 (Pin_1), J4.1 (Pin_1), J40.1 (Pin_1), J43.1 (Pin_1), J47.1 (Pin_1), J7.1 (Pin_1), R3.2, U5.3 (VDD), U6.3 (VDD)
- net ENC1_CS: now also J35.6 (Pin_6)
- net ENC2_CS: now also J40.6 (Pin_6)
- net ENC3_CS: now also J43.6 (Pin_6)
- net ENC4_CS: now also J47.6 (Pin_6)
- net ENC5_A: now also J20.1 (Pin_1)
- net ENC5_B: now also J20.3 (Pin_3)
- net ENC6_A: now also J24.1 (Pin_1)
- net ENC6_B: now also J24.3 (Pin_3)
- net ENC7_A: now also J27.1 (Pin_1)
- net ENC7_B: now also J27.3 (Pin_3)
- net ENC8_A: now also J31.1 (Pin_1)
- net ENC8_B: now also J31.3 (Pin_3)
- net EXT_LED1: now also R2.2
- net EXT_LED2: now also R6.2
- net EXT_LED3: now also R8.2
- net FDCAN1_RX: now also U5.4 (RXD)
- net FDCAN1_TX: now also U5.1 (TXD)
- net FDCAN2_RX: now also U6.4 (RXD)
- net FDCAN2_TX: now also U6.1 (TXD)
- net GND: now also C1.2, C2.2, C3.2, C4.2, D2.1 (K), D3.1 (K), D4.1 (K), D7.1 (K), IC1.2 (CATHODE_1), IC1.3 (CATHODE_2), IC2.2 (CATHODE_1), IC2.3 (CATHODE_2), IC3.2 (CATHODE_1), IC3.3 (CATHODE_2), J11.2 (Pin_2), J12.4 (Pin_4), J13.3 (Pin_3), J14.2 (Pin_2), J18.1 (Pin_1), J19.1 (Pin_1), J20.4 (Pin_4), J22.1 (Pin_1), J23.1 (Pin_1), J24.4 (Pin_4), J25.1 (Pin_1), J26.1 (Pin_1), J27.4 (Pin_4), J29.1 (Pin_1), J3.2 (Pin_2), J30.1 (Pin_1), J31.4 (Pin_4), J34.2 (Pin_2), J35.4 (Pin_4), J36.2 (Pin_2), J37.2 (Pin_2), J39.2 (Pin_2), J4.2 (Pin_2), J40.4 (Pin_4), J41.2 (Pin_2), J42.2 (Pin_2), J43.4 (Pin_4), J44.2 (Pin_2), J45.2 (Pin_2), J46.2 (Pin_2), J47.4 (Pin_4), J48.2 (Pin_2), J7.2 (Pin_2), J8.3 (Pin_3), SW1.3 (C), SW1.6 (C), U1.2, U1.4, U1.6, U1.8, U3.2, U3.4, U4.2, U4.4, U4.6, U4.8, U5.2 (VSS), U5.8 (STBY), U6.2 (VSS), U6.8 (STBY)
- net I2C1_SCL: now also J8.2 (Pin_2), R18.1
- net I2C1_SDA: now also J8.4 (Pin_4), R19.1
- net I2C2_SCL: now also J13.2 (Pin_2), R22.1
- net I2C2_SDA: now also J13.4 (Pin_4), R24.1
- net LIMIT_SW1: now also J34.1 (Pin_1), R40.2
- net LIMIT_SW10: now also J48.1 (Pin_1), R54.2
- net LIMIT_SW11: now also SW1.2 (B)
- net LIMIT_SW12: now also SW1.5 (B)
- net LIMIT_SW2: now also J36.1 (Pin_1), R43.2
- net LIMIT_SW3: now also J37.1 (Pin_1), R44.2
- net LIMIT_SW4: now also J39.1 (Pin_1), R46.2
- net LIMIT_SW5: now also J41.1 (Pin_1), R48.2
- net LIMIT_SW6: now also J42.1 (Pin_1), R50.2
- net LIMIT_SW7: now also J44.1 (Pin_1), R51.2
- net LIMIT_SW8: now also J45.1 (Pin_1), R52.2
- net LIMIT_SW9: now also J46.1 (Pin_1), R53.2
- net M1_PWM1: now also J18.3 (Pin_3)
- net M1_PWM2: now also J18.4 (Pin_4)
- net M2_PWM1: now also J22.3 (Pin_3)
- net M2_PWM2: now also J22.4 (Pin_4)
- net M3_PWM1: now also J25.3 (Pin_3)
- net M3_PWM2: now also J25.4 (Pin_4)
- net M4_PWM1: now also J29.3 (Pin_3)
- net M4_PWM2: now also J29.4 (Pin_4)
- net M5_PWM1: now also J19.3 (Pin_3)
- net M5_PWM2: now also J19.4 (Pin_4)
- net M6_PWM1: now also J23.3 (Pin_3)
- net M6_PWM2: now also J23.4 (Pin_4)
- net M7_PWM1: now also J26.3 (Pin_3)
- net M7_PWM2: now also J26.4 (Pin_4)
- net M8_PWM1: now also J30.3 (Pin_3)
- net M8_PWM2: now also J30.4 (Pin_4)
- net SERVO1: now also IC1.1 (ANODE_1)
- net SERVO2: now also IC1.4 (ANODE_2)
- net SERVO3: now also IC2.1 (ANODE_1)
- net SERVO4: now also IC2.4 (ANODE_2)
- net SERVO5: now also IC3.1 (ANODE_1)
- net SERVO6: now also IC3.4 (ANODE_2)
- net SOLENOID1: now also R1.2
- net SOLENOID10: now also R45.2
- net SOLENOID2: now also R10.2
- net SOLENOID3: now also R15.2
- net SOLENOID4: now also R20.2
- net SOLENOID5: now also R25.2
- net SOLENOID6: now also R28.2
- net SOLENOID7: now also R32.2
- net SOLENOID8: now also R35.2
- net SOLENOID9: now also R39.2
- net SPI1_MISO: now also J35.5 (Pin_5), J40.5 (Pin_5), J43.5 (Pin_5), J47.5 (Pin_5)
- net SPI1_MOSI: now also J35.3 (Pin_3), J40.3 (Pin_3), J43.3 (Pin_3), J47.3 (Pin_3)
- net SPI1_SCK: now also J35.2 (Pin_2), J40.2 (Pin_2), J43.2 (Pin_2), J47.2 (Pin_2)
- net SPI3_MISO: now also J12.5 (Pin_5)
- net SPI3_MOSI: now also J12.3 (Pin_3)
- net SPI3_SCK: now also J12.2 (Pin_2)
- net UART7_RX: now also J14.4 (Pin_4)
- net UART7_TX: now also J14.3 (Pin_3)
- net USART2_RX: now also J7.4 (Pin_4)
- net USART2_TX: now also J7.3 (Pin_3)
- net USART3_RX: now also J11.4 (Pin_4)
- net USART3_TX: now also J11.3 (Pin_3)
- net INT2: now reaches U2.CN12_67 (PG7)
- net INT2: now also J13.5 (Pin_5)
- net INT1: now reaches U2.CN12_70 (PG6)
- net INT1: now also J8.5 (Pin_5)
- new net: D14.2 (A), J28.2 (Pin_2), Q8.3 (D)
- new net: D12.2 (A), J16.2 (Pin_2), Q6.3 (D)
- new net: R20.1, U1.7
- new net: R21.2, U1.9
- new net: Q3.1 (G), R16.1, R17.2
- new net: R39.1, U3.1
- new net: R41.2, U3.15
- new net: IC1.6 (VO2_(OUTPUT_2)), M2.1 (PWM)
- new net: IC1.7 (VO1_(OUTPUT_1)), M1.1 (PWM)
- new net: D8.2 (A), R9.1
- new net: Q7.1 (G), R33.1, R34.2
- new net: D13.2 (A), J21.2 (Pin_2), Q7.3 (D)
- new net: R14.1, SW1.4 (A)
- new net: Q5.1 (G), R26.1, R27.2
- new net: D15.2 (A), J33.2 (Pin_2), Q9.3 (D)
- new net: Q8.1 (G), R36.1, R37.2
- new net: D1.2 (A), J1.2 (Pin_2), Q1.3 (D)
- new net: R35.1, U4.7
- new net: R36.2, U4.9
- new net: IC3.6 (VO2_(OUTPUT_2)), M6.1 (PWM)
- new net: IC3.7 (VO1_(OUTPUT_1)), M5.1 (PWM)
- new net: D6.2 (A), J2.2 (Pin_2), Q2.3 (D)
- new net: Q10.1 (G), R47.1, R49.2
- new net: D16.2 (A), J38.2 (Pin_2), Q10.3 (D)
- new net: R28.1, U4.3
- new net: D10.2 (A), J9.2 (Pin_2), Q4.3 (D)
- new net: R32.1, U4.5
- new net: R16.2, U1.11
- new net: R15.1, U1.5
- new net: R11.2, U1.13
- new net: R10.1, U1.3
- new net: R33.2, U4.11
- new net: D2.2 (A), R2.1
- new net: R1.1, U1.1
- new net: J17.2 (Pin_2), R31.1
- new net: Q2.1 (G), R11.1, R12.2
- new net: D5.2 (A), R7.1
- new net: D9.2 (A), J5.2 (Pin_2), Q3.3 (D)
- new net: D11.2 (A), J15.2 (Pin_2), Q5.3 (D)
- new net: R13.1, SW1.1 (A)
- new net: D7.2 (A), R8.1
- new net: Q1.1 (G), R4.1, R5.2
- new net: R4.2, U1.15
- new net: Q6.1 (G), R29.1, R30.2
- new net: J32.2 (Pin_2), R38.1
- new net: R47.2, U3.13
- new net: Q4.1 (G), R21.1, R23.2
- new net: Q9.1 (G), R41.1, R42.2
- new net: D4.2 (A), R6.1
- new net: IC2.6 (VO2_(OUTPUT_2)), M4.1 (PWM)
- new net: R25.1, U4.1
- new net: R45.1, U3.3
- new net: R26.2, U4.15
- new net: IC2.7 (VO1_(OUTPUT_1)), M3.1 (PWM)
- new net: R29.2, U4.13
- new net: D3.2 (A), R3.1
- new net +24V: D1.1 (K), D10.1 (K), D11.1 (K), D12.1 (K), D13.1 (K), D14.1 (K), D15.1 (K), D16.1 (K), D6.1 (K), D9.1 (K), J1.1 (Pin_1), J15.1 (Pin_1), J16.1 (Pin_1), J2.1 (Pin_1), J21.1 (Pin_1), J28.1 (Pin_1), J33.1 (Pin_1), J38.1 (Pin_1), J49.2 (Pin_2), J5.1 (Pin_1), J50.2 (Pin_2), J9.1 (Pin_1), R7.2, U1.10, U1.12, U1.14, U1.16, U3.14, U3.16, U4.10, U4.12, U4.14, U4.16
- new net +3.3V: C2.1, C4.1, U5.5 (Vio), U6.5 (Vio)
- new net +8V: C5.1, C6.1, C7.1, IC1.8 (VCC), IC2.8 (VCC), IC3.8 (VCC), J51.2 (Pin_2), J52.2 (Pin_2), M1.2 (+), M2.2 (+), M3.2 (+), M4.2 (+), M5.2 (+), M6.2 (+), R9.2
- new net FDCAN1_H: J17.1 (Pin_1), J6.1 (Pin_1), U5.7 (CANH)
- new net FDCAN1_L: J6.2 (Pin_2), R31.2, U5.6 (CANL)
- new net FDCAN2_H: J10.1 (Pin_1), J32.1 (Pin_1), U6.7 (CANH)
- new net FDCAN2_L: J10.2 (Pin_2), R38.2, U6.6 (CANL)
- new net GND2: C5.2, C6.2, C7.2, D5.1 (K), D8.1 (K), IC1.5 (GND), IC2.5 (GND), IC3.5 (GND), J49.1 (Pin_1), J50.1 (Pin_1), J51.1 (Pin_1), J52.1 (Pin_1), M1.3 (-), M2.3 (-), M3.3 (-), M4.3 (-), M5.3 (-), M6.3 (-), Q1.2 (S), Q10.2 (S), Q2.2 (S), Q3.2 (S), Q4.2 (S), Q5.2 (S), Q6.2 (S), Q7.2 (S), Q8.2 (S), Q9.2 (S), R12.1, R17.1, R23.1, R27.1, R30.1, R34.1, R37.1, R42.1, R49.1, R5.1
Other:
- moved on the sheet: U2A, U2B, U2I, U2J
